Commit message: leave now, cache everythings

File: ros2_ws/src/mentor_pi_hardwares/config/ackermann/description.urdf.xacro (robot description, xacro)
@@ -2,5 +2,11 @@
 <robot name="mentor_pi_ackermann" xmlns:xacro="http://www.ros.org/wiki/xacro">
   <xacro:macro name="ackermann_car" params="">
+    <link name="rear_axle_footprint"/>
     <link name="base_footprint"/>
+    <joint name="rear_axle_footprint_joint" type="fixed">
+      <parent link="rear_axle_footprint"/>
+      <child link="base_footprint"/>
+      <origin xyz="0.0675 0 0" rpy="0 0 0"/>
+    </joint>
     <link name="base_link">
       <inertial>

File: ros2_ws/src/mentor_pi_hardwares/config/ackermann/mentor_pi.urdf.xacro (robot description, xacro)
@@ -8,10 +8,10 @@
   <xacro:arg name="steering_pwm_center_us" default="1500"/>
   <xacro:arg name="steering_pwm_max_us" default="2500"/>
-  <xacro:arg name="steering_angle_min_rad" default="-1.5"/>
-  <xacro:arg name="steering_angle_max_rad" default="1.5"/>
+  <xacro:arg name="steering_angle_min_rad" default="-0.6"/>
+  <xacro:arg name="steering_angle_max_rad" default="0.6"/>
   <xacro:arg name="steering_inverted" default="true"/>
   <xacro:arg name="steering_duration_ms" default="20"/>
-  <xacro:arg name="rear_wheel_radius_m" default="0.0333"/>
-  <xacro:arg name="wheelbase_m" default="0.145"/>
+  <xacro:arg name="rear_wheel_radius_m" default="0.0325"/>
+  <xacro:arg name="wheelbase_m" default="0.135"/>
   <xacro:arg name="linear_adrc_input_gain_per_second" default="5.0"/>
   <xacro:arg name="linear_adrc_controller_bandwidth_rad_s" default="1.0"/>

File: ros2_ws/src/mentor_pi_hardwares/config/ackermann/ros2_control.xacro (robot description, xacro)
@@ -2,5 +2,5 @@
 <robot xmlns:xacro="http://www.ros.org/wiki/xacro">
   <xacro:macro name="ackermann_control"
-               params="robot_name:=mentor_pi feedback_timeout_ms:=100 imu_timeout_ms:=100 steering_pwm_channel:=3 steering_pwm_min_us:=500 steering_pwm_center_us:=1500 steering_pwm_max_us:=2500 steering_angle_min_rad:=-1.5 steering_angle_max_rad:=1.5 steering_inverted:=true steering_duration_ms:=20 rear_wheel_radius_m:=0.0333 wheelbase_m:=0.145 linear_adrc_input_gain_per_second:=5.0 linear_adrc_controller_bandwidth_rad_s:=1.0 linear_adrc_observer_bandwidth_rad_s:=3.0 yaw_adrc_input_gain_per_mps:=30.0 yaw_adrc_controller_bandwidth_rad_s:=1.0 yaw_adrc_observer_bandwidth_rad_s:=3.0 yaw_adrc_minimum_speed_mps:=0.1">
+               params="robot_name:=mentor_pi feedback_timeout_ms:=100 imu_timeout_ms:=100 steering_pwm_channel:=3 steering_pwm_min_us:=500 steering_pwm_center_us:=1500 steering_pwm_max_us:=2500 steering_angle_min_rad:=-0.6 steering_angle_max_rad:=0.6 steering_inverted:=true steering_duration_ms:=20 rear_wheel_radius_m:=0.0325 wheelbase_m:=0.135 linear_adrc_input_gain_per_second:=5.0 linear_adrc_controller_bandwidth_rad_s:=1.0 linear_adrc_observer_bandwidth_rad_s:=3.0 yaw_adrc_input_gain_per_mps:=30.0 yaw_adrc_controller_bandwidth_rad_s:=1.0 yaw_adrc_observer_bandwidth_rad_s:=3.0 yaw_adrc_minimum_speed_mps:=0.1">
     <ros2_control name="mentor_pi_hardware" type="system">
       <hardware>

Commit message: simulator

File: ros2_ws/src/mentor_pi_hardwares/config/ackermann/description.urdf.xacro (robot description, xacro)
@@ -5,7 +5,7 @@
     <link name="base_footprint"/>
     <joint name="rear_axle_footprint_joint" type="fixed">
-      <parent link="rear_axle_footprint"/>
-      <child link="base_footprint"/>
-      <origin xyz="0.0675 0 0" rpy="0 0 0"/>
+      <parent link="base_footprint"/>
+      <child link="rear_axle_footprint"/>
+      <origin xyz="-0.0675 0 0" rpy="0 0 0"/>
     </joint>
     <link name="base_link">

Commit message: Namespace robot description frames

File: ros2_ws/src/mentor_pi_hardwares/config/ackermann/description.urdf.xacro (robot description, xacro)
@@ -1,13 +1,13 @@
 <?xml version="1.0"?>
 <robot name="mentor_pi_ackermann" xmlns:xacro="http://www.ros.org/wiki/xacro">
-  <xacro:macro name="ackermann_car" params="">
-    <link name="rear_axle_footprint"/>
-    <link name="base_footprint"/>
+  <xacro:macro name="ackermann_car" params="frame_prefix:=''">
+    <link name="${frame_prefix}rear_axle_footprint"/>
+    <link name="${frame_prefix}base_footprint"/>
     <joint name="rear_axle_footprint_joint" type="fixed">
-      <parent link="base_footprint"/>
-      <child link="rear_axle_footprint"/>
+      <parent link="${frame_prefix}base_footprint"/>
+      <child link="${frame_prefix}rear_axle_footprint"/>
       <origin xyz="-0.0675 0 0" rpy="0 0 0"/>
     </joint>
-    <link name="base_link">
+    <link name="${frame_prefix}base_link">
       <inertial>
         <origin xyz="0 0 0.025" rpy="0 0 0"/>
@@ -27,54 +27,54 @@
     </link>
     <joint name="base_footprint_joint" type="fixed">
-      <parent link="base_footprint"/>
-      <child link="base_link"/>
+      <parent link="${frame_prefix}base_footprint"/>
+      <child link="${frame_prefix}base_link"/>
       <origin xyz="0 0 0" rpy="0 0 0"/>
     </joint>
-    <link name="wheel_left_front_link">
+    <link name="${frame_prefix}wheel_left_front_link">
       <visual><geometry><cylinder radius="0.04" length="0.02"/></geometry></visual>
       <collision><geometry><cylinder radius="0.04" length="0.02"/></geometry></collision>
     </link>
     <joint name="wheel_left_front_joint" type="revolute">
-      <parent link="base_link"/>
-      <child link="wheel_left_front_link"/>
+      <parent link="${frame_prefix}base_link"/>
+      <child link="${frame_prefix}wheel_left_front_link"/>
       <origin xyz="0.11 0.09 -0.03" rpy="0 0 0"/>
       <axis xyz="0 0 1"/>
       <limit lower="-0.6" upper="0.6" effort="1.0" velocity="1.5"/>
     </joint>
-    <link name="wheel_right_front_link">
+    <link name="${frame_prefix}wheel_right_front_link">
       <visual><geometry><cylinder radius="0.04" length="0.02"/></geometry></visual>
       <collision><geometry><cylinder radius="0.04" length="0.02"/></geometry></collision>
     </link>
     <joint name="wheel_right_front_joint" type="revolute">
-      <parent link="base_link"/>
-      <child link="wheel_right_front_link"/>
+      <parent link="${frame_prefix}base_link"/>
+      <child link="${frame_prefix}wheel_right_front_link"/>
       <origin xyz="0.11 -0.09 -0.03" rpy="0 0 0"/>
       <axis xyz="0 0 1"/>
       <limit lower="-0.6" upper="0.6" effort="1.0" velocity="1.5"/>
     </joint>
-    <link name="wheel_left_rear_link">
+    <link name="${frame_prefix}wheel_left_rear_link">
       <visual><geometry><cylinder radius="0.04" length="0.02"/></geometry></visual>
       <collision><geometry><cylinder radius="0.04" length="0.02"/></geometry></collision>
     </link>
     <joint name="wheel_left_rear_joint" type="continuous">
-      <parent link="base_link"/>
-      <child link="wheel_left_rear_link"/>
+      <parent link="${frame_prefix}base_link"/>
+      <child link="${frame_prefix}wheel_left_rear_link"/>
       <origin xyz="-0.11 0.09 -0.03" rpy="0 0 0"/>
       <axis xyz="0 1 0"/>
     </joint>
-    <link name="wheel_right_rear_link">
+    <link name="${frame_prefix}wheel_right_rear_link">
       <visual><geometry><cylinder radius="0.04" length="0.02"/></geometry></visual>
       <collision><geometry><cylinder radius="0.04" length="0.02"/></geometry></collision>
     </link>
     <joint name="wheel_right_rear_joint" type="continuous">
-      <parent link="base_link"/>
-      <child link="wheel_right_rear_link"/>
+      <parent link="${frame_prefix}base_link"/>
+      <child link="${frame_prefix}wheel_right_rear_link"/>
       <origin xyz="-0.11 -0.09 -0.03" rpy="0 0 0"/>
       <axis xyz="0 1 0"/>
     </joint>
-    <link name="imu_link"/>
+    <link name="${frame_prefix}imu_link"/>
     <joint name="imu_joint" type="fixed">
-      <parent link="base_link"/>
-      <child link="imu_link"/>
+      <parent link="${frame_prefix}base_link"/>
+      <child link="${frame_prefix}imu_link"/>
       <origin xyz="0 0 0.05" rpy="0 0 0"/>
     </joint>

File: ros2_ws/src/mentor_pi_hardwares/config/ackermann/mentor_pi.urdf.xacro (robot description, xacro)
@@ -25,5 +25,5 @@
   <xacro:include filename="$(find mentor_pi_hardwares)/config/ackermann/description.urdf.xacro"/>
   <xacro:include filename="$(find mentor_pi_hardwares)/config/ackermann/ros2_control.xacro"/>
-  <xacro:ackermann_car/>
+  <xacro:ackermann_car frame_prefix="$(arg robot_name)/"/>
   <xacro:ackermann_control
       robot_name="$(arg robot_name)"

File: ros2_ws/src/mentor_pi_hardwares/config/ackermann/simulation.urdf.xacro (robot description, xacro)
@@ -4,5 +4,5 @@
   <xacro:include filename="$(find mentor_pi_hardwares)/config/ackermann/description.urdf.xacro"/>
   <xacro:include filename="$(find mentor_pi_hardwares)/config/ackermann/simulation_ros2_control.xacro"/>
-  <xacro:ackermann_car/>
+  <xacro:ackermann_car frame_prefix="$(arg robot_name)/"/>
   <xacro:ackermann_simulation_control robot_name="$(arg robot_name)"/>
 </robot>

File: ros2_ws/src/mentor_pi_hardwares/config/mecanum/description.urdf.xacro (robot description, xacro)
@@ -1,7 +1,7 @@
 <?xml version="1.0"?>
 <robot name="mentor_pi_mecanum" xmlns:xacro="http://www.ros.org/wiki/xacro">
-  <xacro:macro name="mecanum_car" params="">
-    <link name="base_footprint"/>
-    <link name="base_link">
+  <xacro:macro name="mecanum_car" params="frame_prefix:=''">
+    <link name="${frame_prefix}base_footprint"/>
+    <link name="${frame_prefix}base_link">
       <inertial>
         <origin xyz="0 0 0.025" rpy="0 0 0"/>
@@ -21,52 +21,52 @@
     </link>
     <joint name="base_footprint_joint" type="fixed">
-      <parent link="base_footprint"/>
-      <child link="base_link"/>
+      <parent link="${frame_prefix}base_footprint"/>
+      <child link="${frame_prefix}base_link"/>
       <origin xyz="0 0 0" rpy="0 0 0"/>
     </joint>
-    <link name="wheel_left_front_link">
+    <link name="${frame_prefix}wheel_left_front_link">
       <visual><geometry><cylinder radius="0.04" length="0.02"/></geometry></visual>
       <collision><geometry><cylinder radius="0.04" length="0.02"/></geometry></collision>
     </link>
     <joint name="wheel_left_front_joint" type="continuous">
-      <parent link="base_link"/>
-      <child link="wheel_left_front_link"/>
+      <parent link="${frame_prefix}base_link"/>
+      <child link="${frame_prefix}wheel_left_front_link"/>
       <origin xyz="0.11 0.09 -0.03" rpy="0 0 0"/>
       <axis xyz="0 1 0"/>
     </joint>
-    <link name="wheel_right_front_link">
+    <link name="${frame_prefix}wheel_right_front_link">
       <visual><geometry><cylinder radius="0.04" length="0.02"/></geometry></visual>
       <collision><geometry><cylinder radius="0.04" length="0.02"/></geometry></collision>
     </link>
     <joint name="wheel_right_front_joint" type="continuous">
-      <parent link="base_link"/>
-      <child link="wheel_right_front_link"/>
+      <parent link="${frame_prefix}base_link"/>
+      <child link="${frame_prefix}wheel_right_front_link"/>
       <origin xyz="0.11 -0.09 -0.03" rpy="0 0 0"/>
       <axis xyz="0 1 0"/>
     </joint>
-    <link name="wheel_left_rear_link">
+    <link name="${frame_prefix}wheel_left_rear_link">
       <visual><geometry><cylinder radius="0.04" length="0.02"/></geometry></visual>
       <collision><geometry><cylinder radius="0.04" length="0.02"/></geometry></collision>
     </link>
     <joint name="wheel_left_rear_joint" type="continuous">
-      <parent link="base_link"/>
-      <child link="wheel_left_rear_link"/>
+      <parent link="${frame_prefix}base_link"/>
+      <child link="${frame_prefix}wheel_left_rear_link"/>
       <origin xyz="-0.11 0.09 -0.03" rpy="0 0 0"/>
       <axis xyz="0 1 0"/>
     </joint>
-    <link name="wheel_right_rear_link">
+    <link name="${frame_prefix}wheel_right_rear_link">
       <visual><geometry><cylinder radius="0.04" length="0.02"/></geometry></visual>
       <collision><geometry><cylinder radius="0.04" length="0.02"/></geometry></collision>
     </link>
     <joint name="wheel_right_rear_joint" type="continuous">
-      <parent link="base_link"/>
-      <child link="wheel_right_rear_link"/>
+      <parent link="${frame_prefix}base_link"/>
+      <child link="${frame_prefix}wheel_right_rear_link"/>
       <origin xyz="-0.11 -0.09 -0.03" rpy="0 0 0"/>
       <axis xyz="0 1 0"/>
     </joint>
-    <link name="imu_link"/>
+    <link name="${frame_prefix}imu_link"/>
     <joint name="imu_joint" type="fixed">
-      <parent link="base_link"/>
-      <child link="imu_link"/>
+      <parent link="${frame_prefix}base_link"/>
+      <child link="${frame_prefix}imu_link"/>
       <origin xyz="0 0 0.05" rpy="0 0 0"/>
     </joint>

File: ros2_ws/src/mentor_pi_hardwares/config/mecanum/mentor_pi.urdf.xacro (robot description, xacro)
@@ -16,5 +16,5 @@
   <xacro:include filename="$(find mentor_pi_hardwares)/config/mecanum/description.urdf.xacro"/>
   <xacro:include filename="$(find mentor_pi_hardwares)/config/mecanum/ros2_control.xacro"/>
-  <xacro:mecanum_car/>
+  <xacro:mecanum_car frame_prefix="$(arg robot_name)/"/>
   <xacro:mecanum_control robot_name="$(arg robot_name)"
                          feedback_timeout_ms="$(arg feedback_timeout_ms)"

File: ros2_ws/src/mentor_pi_hardwares/config/mecanum/simulation.urdf.xacro (robot description, xacro)
@@ -4,5 +4,5 @@
   <xacro:include filename="$(find mentor_pi_hardwares)/config/mecanum/description.urdf.xacro"/>
   <xacro:include filename="$(find mentor_pi_hardwares)/config/mecanum/simulation_ros2_control.xacro"/>
-  <xacro:mecanum_car/>
+  <xacro:mecanum_car frame_prefix="$(arg robot_name)/"/>
   <xacro:mecanum_simulation_control robot_name="$(arg robot_name)"/>
 </robot>

Commit message: Restore Mentor Pi mesh visuals

File: ros2_ws/src/mentor_pi_hardwares/config/ackermann/description.urdf.xacro (robot description, xacro)
@@ -1,4 +1,10 @@
 <?xml version="1.0"?>
 <robot name="mentor_pi_ackermann" xmlns:xacro="http://www.ros.org/wiki/xacro">
+  <material name="mentor_pi_gray">
+    <color rgba="0.7 0.7 0.7 1.0"/>
+  </material>
+  <material name="mentor_pi_black">
+    <color rgba="0.1 0.1 0.1 1.0"/>
+  </material>
   <xacro:macro name="ackermann_car" params="frame_prefix:=''">
     <link name="${frame_prefix}rear_axle_footprint"/>
@@ -16,7 +22,23 @@
       </inertial>
       <visual>
+        <origin xyz="0 0 0.070" rpy="-1.5707963267948966 0 0"/>
         <geometry>
-          <box size="0.22 0.16 0.06"/>
+          <mesh filename="package://mentor_pi_hardwares/config/ackermann/meshes/base_link.stl"/>
         </geometry>
+        <material name="mentor_pi_gray"/>
+      </visual>
+      <visual>
+        <origin xyz="0.064015 -0.00013463 0.121155" rpy="-1.5707963267948966 0 0"/>
+        <geometry>
+          <mesh filename="package://mentor_pi_hardwares/config/ackermann/meshes/cam_link.stl"/>
+        </geometry>
+        <material name="mentor_pi_black"/>
+      </visual>
+      <visual>
+        <origin xyz="-0.0096019 -0.00008533 0.162501" rpy="-1.5707963267948966 0 0"/>
+        <geometry>
+          <mesh filename="package://mentor_pi_hardwares/config/ackermann/meshes/lidar_link.stl"/>
+        </geometry>
+        <material name="mentor_pi_black"/>
       </visual>
       <collision>
@@ -32,5 +54,10 @@
     </joint>
     <link name="${frame_prefix}wheel_left_front_link">
-      <visual><geometry><cylinder radius="0.04" length="0.02"/></geometry></visual>
+      <visual>
+        <geometry>
+          <mesh filename="package://mentor_pi_hardwares/config/ackermann/meshes/wheel_left_front_link.stl"/>
+        </geometry>
+        <material name="mentor_pi_black"/>
+      </visual>
       <collision><geometry><cylinder radius="0.04" length="0.02"/></geometry></collision>
     </link>
@@ -38,10 +65,15 @@
       <parent link="${frame_prefix}base_link"/>
       <child link="${frame_prefix}wheel_left_front_link"/>
-      <origin xyz="0.11 0.09 -0.03" rpy="0 0 0"/>
+      <origin xyz="0.0675 0.070 0.0325" rpy="0 0 0"/>
       <axis xyz="0 0 1"/>
       <limit lower="-0.6" upper="0.6" effort="1.0" velocity="1.5"/>
     </joint>
     <link name="${frame_prefix}wheel_right_front_link">
-      <visual><geometry><cylinder radius="0.04" length="0.02"/></geometry></visual>
+      <visual>
+        <geometry>
+          <mesh filename="package://mentor_pi_hardwares/config/ackermann/meshes/wheel_right_front_link.stl"/>
+        </geometry>
+        <material name="mentor_pi_black"/>
+      </visual>
       <collision><geometry><cylinder radius="0.04" length="0.02"/></geometry></collision>
     </link>
@@ -49,10 +81,15 @@
       <parent link="${frame_prefix}base_link"/>
       <child link="${frame_prefix}wheel_right_front_link"/>
-      <origin xyz="0.11 -0.09 -0.03" rpy="0 0 0"/>
+      <origin xyz="0.0675 -0.070 0.0325" rpy="0 0 0"/>
       <axis xyz="0 0 1"/>
       <limit lower="-0.6" upper="0.6" effort="1.0" velocity="1.5"/>
     </joint>
     <link name="${frame_prefix}wheel_left_rear_link">
-      <visual><geometry><cylinder radius="0.04" length="0.02"/></geometry></visual>
+      <visual>
+        <geometry>
+          <mesh filename="package://mentor_pi_hardwares/config/ackermann/meshes/wheel_left_rear_link.stl"/>
+        </geometry>
+        <material name="mentor_pi_black"/>
+      </visual>
       <collision><geometry><cylinder radius="0.04" length="0.02"/></geometry></collision>
     </link>
@@ -60,9 +97,14 @@
       <parent link="${frame_prefix}base_link"/>
       <child link="${frame_prefix}wheel_left_rear_link"/>
-      <origin xyz="-0.11 0.09 -0.03" rpy="0 0 0"/>
+      <origin xyz="-0.0675 0.070 0.0325" rpy="0 0 0"/>
       <axis xyz="0 1 0"/>
     </joint>
     <link name="${frame_prefix}wheel_right_rear_link">
-      <visual><geometry><cylinder radius="0.04" length="0.02"/></geometry></visual>
+      <visual>
+        <geometry>
+          <mesh filename="package://mentor_pi_hardwares/config/ackermann/meshes/wheel_right_rear_link.stl"/>
+        </geometry>
+        <material name="mentor_pi_black"/>
+      </visual>
       <collision><geometry><cylinder radius="0.04" length="0.02"/></geometry></collision>
     </link>
@@ -70,5 +112,5 @@
       <parent link="${frame_prefix}base_link"/>
       <child link="${frame_prefix}wheel_right_rear_link"/>
-      <origin xyz="-0.11 -0.09 -0.03" rpy="0 0 0"/>
+      <origin xyz="-0.0675 -0.070 0.0325" rpy="0 0 0"/>
       <axis xyz="0 1 0"/>
     </joint>

File: ros2_ws/src/mentor_pi_hardwares/config/mecanum/description.urdf.xacro (robot description, xacro)
@@ -1,4 +1,10 @@
 <?xml version="1.0"?>
 <robot name="mentor_pi_mecanum" xmlns:xacro="http://www.ros.org/wiki/xacro">
+  <material name="mentor_pi_gray">
+    <color rgba="0.7 0.7 0.7 1.0"/>
+  </material>
+  <material name="mentor_pi_black">
+    <color rgba="0.1 0.1 0.1 1.0"/>
+  </material>
   <xacro:macro name="mecanum_car" params="frame_prefix:=''">
     <link name="${frame_prefix}base_footprint"/>
@@ -10,7 +16,23 @@
       </inertial>
       <visual>
+        <origin xyz="0 0 0.050" rpy="-1.5707963267948966 0 0"/>
         <geometry>
-          <box size="0.22 0.16 0.06"/>
+          <mesh filename="package://mentor_pi_hardwares/config/mecanum/meshes/base_link.stl"/>
         </geometry>
+        <material name="mentor_pi_gray"/>
+      </visual>
+      <visual>
+        <origin xyz="0.064015 -0.00013463 0.101155" rpy="-1.5707963267948966 0 0"/>
+        <geometry>
+          <mesh filename="package://mentor_pi_hardwares/config/mecanum/meshes/cam_link.stl"/>
+        </geometry>
+        <material name="mentor_pi_black"/>
+      </visual>
+      <visual>
+        <origin xyz="-0.0096019 -0.00008533 0.142501" rpy="-1.5707963267948966 0 0"/>
+        <geometry>
+          <mesh filename="package://mentor_pi_hardwares/config/mecanum/meshes/lidar_link.stl"/>
+        </geometry>
+        <material name="mentor_pi_black"/>
       </visual>
       <collision>
@@ -26,5 +48,10 @@
     </joint>
     <link name="${frame_prefix}wheel_left_front_link">
-      <visual><geometry><cylinder radius="0.04" length="0.02"/></geometry></visual>
+      <visual>
+        <geometry>
+          <mesh filename="package://mentor_pi_hardwares/config/mecanum/meshes/wheel_left_front_link.stl"/>
+        </geometry>
+        <material name="mentor_pi_black"/>
+      </visual>
       <collision><geometry><cylinder radius="0.04" length="0.02"/></geometry></collision>
     </link>
@@ -32,9 +59,14 @@
       <parent link="${frame_prefix}base_link"/>
       <child link="${frame_prefix}wheel_left_front_link"/>
-      <origin xyz="0.11 0.09 -0.03" rpy="0 0 0"/>
+      <origin xyz="0.065812864 0.074187136 0.0325" rpy="0 0 0"/>
       <axis xyz="0 1 0"/>
     </joint>
     <link name="${frame_prefix}wheel_right_front_link">
-      <visual><geometry><cylinder radius="0.04" length="0.02"/></geometry></visual>
+      <visual>
+        <geometry>
+          <mesh filename="package://mentor_pi_hardwares/config/mecanum/meshes/wheel_right_front_link.stl"/>
+        </geometry>
+        <material name="mentor_pi_black"/>
+      </visual>
       <collision><geometry><cylinder radius="0.04" length="0.02"/></geometry></collision>
     </link>
@@ -42,9 +74,14 @@
       <parent link="${frame_prefix}base_link"/>
       <child link="${frame_prefix}wheel_right_front_link"/>
-      <origin xyz="0.11 -0.09 -0.03" rpy="0 0 0"/>
+      <origin xyz="0.065812864 -0.074187136 0.0325" rpy="0 0 0"/>
       <axis xyz="0 1 0"/>
     </joint>
     <link name="${frame_prefix}wheel_left_rear_link">
-      <visual><geometry><cylinder radius="0.04" length="0.02"/></geometry></visual>
+      <visual>
+        <geometry>
+          <mesh filename="package://mentor_pi_hardwares/config/mecanum/meshes/wheel_left_rear_link.stl"/>
+        </geometry>
+        <material name="mentor_pi_black"/>
+      </visual>
       <collision><geometry><cylinder radius="0.04" length="0.02"/></geometry></collision>
     </link>
@@ -52,9 +89,14 @@
       <parent link="${frame_prefix}base_link"/>
       <child link="${frame_prefix}wheel_left_rear_link"/>
-      <origin xyz="-0.11 0.09 -0.03" rpy="0 0 0"/>
+      <origin xyz="-0.065812864 0.074187136 0.0325" rpy="0 0 0"/>
       <axis xyz="0 1 0"/>
     </joint>
     <link name="${frame_prefix}wheel_right_rear_link">
-      <visual><geometry><cylinder radius="0.04" length="0.02"/></geometry></visual>
+      <visual>
+        <geometry>
+          <mesh filename="package://mentor_pi_hardwares/config/mecanum/meshes/wheel_right_rear_link.stl"/>
+        </geometry>
+        <material name="mentor_pi_black"/>
+      </visual>
       <collision><geometry><cylinder radius="0.04" length="0.02"/></geometry></collision>
     </link>
@@ -62,5 +104,5 @@
       <parent link="${frame_prefix}base_link"/>
       <child link="${frame_prefix}wheel_right_rear_link"/>
-      <origin xyz="-0.11 -0.09 -0.03" rpy="0 0 0"/>
+      <origin xyz="-0.065812864 -0.074187136 0.0325" rpy="0 0 0"/>
       <axis xyz="0 1 0"/>
     </joint>
