Commit message: Correct wheel mesh orientation

File: ros2_ws/src/mentor_pi_hardwares/config/ackermann/description.urdf.xacro (robot description, xacro)
@@ -55,4 +55,5 @@
     <link name="${frame_prefix}wheel_left_front_link">
       <visual>
+        <origin xyz="0 0 0" rpy="-1.5707963267948966 0 0"/>
         <geometry>
           <mesh filename="package://mentor_pi_hardwares/config/ackermann/meshes/wheel_left_front_link.stl"/>
@@ -60,5 +61,8 @@
         <material name="mentor_pi_black"/>
       </visual>
-      <collision><geometry><cylinder radius="0.04" length="0.02"/></geometry></collision>
+      <collision>
+        <origin xyz="0 0 0" rpy="-1.5707963267948966 0 0"/>
+        <geometry><cylinder radius="0.04" length="0.02"/></geometry>
+      </collision>
     </link>
     <joint name="wheel_left_front_joint" type="revolute">
@@ -71,4 +75,5 @@
     <link name="${frame_prefix}wheel_right_front_link">
       <visual>
+        <origin xyz="0 0 0" rpy="-1.5707963267948966 0 0"/>
         <geometry>
           <mesh filename="package://mentor_pi_hardwares/config/ackermann/meshes/wheel_right_front_link.stl"/>
@@ -76,5 +81,8 @@
         <material name="mentor_pi_black"/>
       </visual>
-      <collision><geometry><cylinder radius="0.04" length="0.02"/></geometry></collision>
+      <collision>
+        <origin xyz="0 0 0" rpy="-1.5707963267948966 0 0"/>
+        <geometry><cylinder radius="0.04" length="0.02"/></geometry>
+      </collision>
     </link>
     <joint name="wheel_right_front_joint" type="revolute">
@@ -87,4 +95,5 @@
     <link name="${frame_prefix}wheel_left_rear_link">
       <visual>
+        <origin xyz="0 0 0" rpy="-1.5707963267948966 0 0"/>
         <geometry>
           <mesh filename="package://mentor_pi_hardwares/config/ackermann/meshes/wheel_left_rear_link.stl"/>
@@ -92,5 +101,8 @@
         <material name="mentor_pi_black"/>
       </visual>
-      <collision><geometry><cylinder radius="0.04" length="0.02"/></geometry></collision>
+      <collision>
+        <origin xyz="0 0 0" rpy="-1.5707963267948966 0 0"/>
+        <geometry><cylinder radius="0.04" length="0.02"/></geometry>
+      </collision>
     </link>
     <joint name="wheel_left_rear_joint" type="continuous">
@@ -102,4 +114,5 @@
     <link name="${frame_prefix}wheel_right_rear_link">
       <visual>
+        <origin xyz="0 0 0" rpy="-1.5707963267948966 0 0"/>
         <geometry>
           <mesh filename="package://mentor_pi_hardwares/config/ackermann/meshes/wheel_right_rear_link.stl"/>
@@ -107,5 +120,8 @@
         <material name="mentor_pi_black"/>
       </visual>
-      <collision><geometry><cylinder radius="0.04" length="0.02"/></geometry></collision>
+      <collision>
+        <origin xyz="0 0 0" rpy="-1.5707963267948966 0 0"/>
+        <geometry><cylinder radius="0.04" length="0.02"/></geometry>
+      </collision>
     </link>
     <joint name="wheel_right_rear_joint" type="continuous">

File: ros2_ws/src/mentor_pi_hardwares/config/mecanum/description.urdf.xacro (robot description, xacro)
@@ -49,4 +49,5 @@
     <link name="${frame_prefix}wheel_left_front_link">
       <visual>
+        <origin xyz="0 0 0" rpy="-1.5707963267948966 0 0"/>
         <geometry>
           <mesh filename="package://mentor_pi_hardwares/config/mecanum/meshes/wheel_left_front_link.stl"/>
@@ -54,5 +55,8 @@
         <material name="mentor_pi_black"/>
       </visual>
-      <collision><geometry><cylinder radius="0.04" length="0.02"/></geometry></collision>
+      <collision>
+        <origin xyz="0 0 0" rpy="-1.5707963267948966 0 0"/>
+        <geometry><cylinder radius="0.04" length="0.02"/></geometry>
+      </collision>
     </link>
     <joint name="wheel_left_front_joint" type="continuous">
@@ -64,4 +68,5 @@
     <link name="${frame_prefix}wheel_right_front_link">
       <visual>
+        <origin xyz="0 0 0" rpy="-1.5707963267948966 0 0"/>
         <geometry>
           <mesh filename="package://mentor_pi_hardwares/config/mecanum/meshes/wheel_right_front_link.stl"/>
@@ -69,5 +74,8 @@
         <material name="mentor_pi_black"/>
       </visual>
-      <collision><geometry><cylinder radius="0.04" length="0.02"/></geometry></collision>
+      <collision>
+        <origin xyz="0 0 0" rpy="-1.5707963267948966 0 0"/>
+        <geometry><cylinder radius="0.04" length="0.02"/></geometry>
+      </collision>
     </link>
     <joint name="wheel_right_front_joint" type="continuous">
@@ -79,4 +87,5 @@
     <link name="${frame_prefix}wheel_left_rear_link">
       <visual>
+        <origin xyz="0 0 0" rpy="-1.5707963267948966 0 0"/>
         <geometry>
           <mesh filename="package://mentor_pi_hardwares/config/mecanum/meshes/wheel_left_rear_link.stl"/>
@@ -84,5 +93,8 @@
         <material name="mentor_pi_black"/>
       </visual>
-      <collision><geometry><cylinder radius="0.04" length="0.02"/></geometry></collision>
+      <collision>
+        <origin xyz="0 0 0" rpy="-1.5707963267948966 0 0"/>
+        <geometry><cylinder radius="0.04" length="0.02"/></geometry>
+      </collision>
     </link>
     <joint name="wheel_left_rear_joint" type="continuous">
@@ -94,4 +106,5 @@
     <link name="${frame_prefix}wheel_right_rear_link">
       <visual>
+        <origin xyz="0 0 0" rpy="-1.5707963267948966 0 0"/>
         <geometry>
           <mesh filename="package://mentor_pi_hardwares/config/mecanum/meshes/wheel_right_rear_link.stl"/>
@@ -99,5 +112,8 @@
         <material name="mentor_pi_black"/>
       </visual>
-      <collision><geometry><cylinder radius="0.04" length="0.02"/></geometry></collision>
+      <collision>
+        <origin xyz="0 0 0" rpy="-1.5707963267948966 0 0"/>
+        <geometry><cylinder radius="0.04" length="0.02"/></geometry>
+      </collision>
     </link>
     <joint name="wheel_right_rear_joint" type="continuous">
